File: ecad/le-board.kicad_pcb (KiCad board)
At the start: 2 copper layers, 0 parts

Commit message: Added initial placement for MX switches
Parts:
- added D1: 1n4148, Diode_SMD:D_SOD-123, B.Cu at (43.2, 41.1)
- added D10: 1n4148, Diode_SMD:D_SOD-123, B.Cu at (274.0, 41.1)
- added D11: 1n4148, Diode_SMD:D_SOD-123, B.Cu at (43.2, 60.2)
- added D12: 1n4148, Diode_SMD:D_SOD-123, B.Cu at (62.2, 60.2)
- added D13: 1n4148, Diode_SMD:D_SOD-123, B.Cu at (81.3, 60.2)
- added D14: 1n4148, Diode_SMD:D_SOD-123, B.Cu at (100.3, 60.2)
- added D15: 1n4148, Diode_SMD:D_SOD-123, B.Cu at (119.4, 60.2)
- added D16: 1n4148, Diode_SMD:D_SOD-123, B.Cu at (197.8, 60.2)
- added D17: 1n4148, Diode_SMD:D_SOD-123, B.Cu at (216.8, 60.2)
- added D18: 1n4148, Diode_SMD:D_SOD-123, B.Cu at (235.9, 60.2)
- added D19: 1n4148, Diode_SMD:D_SOD-123, B.Cu at (254.9, 60.2)
- added D2: 1n4148, Diode_SMD:D_SOD-123, B.Cu at (62.2, 41.1)
- added D20: 1n4148, Diode_SMD:D_SOD-123, B.Cu at (274.0, 60.2)
- added D21: 1n4148, Diode_SMD:D_SOD-123, B.Cu at (43.2, 79.2)
- added D22: 1n4148, Diode_SMD:D_SOD-123, B.Cu at (62.2, 79.2)
- added D23: 1n4148, Diode_SMD:D_SOD-123, B.Cu at (81.3, 79.2)
- added D24: 1n4148, Diode_SMD:D_SOD-123, B.Cu at (100.3, 79.2)
- added D25: 1n4148, Diode_SMD:D_SOD-123, B.Cu at (119.4, 79.2)
- added D26: 1n4148, Diode_SMD:D_SOD-123, B.Cu at (197.8, 79.2)
- added D27: 1n4148, Diode_SMD:D_SOD-123, B.Cu at (216.8, 79.2)
- added D28: 1n4148, Diode_SMD:D_SOD-123, B.Cu at (235.9, 79.2)
- added D29: 1n4148, Diode_SMD:D_SOD-123, B.Cu at (254.9, 79.2)
- added D3: 1n4148, Diode_SMD:D_SOD-123, B.Cu at (81.3, 41.1)
- added D30: 1n4148, Diode_SMD:D_SOD-123, B.Cu at (274.0, 79.2)
- added D31: 1n4148, Diode_SMD:D_SOD-123, B.Cu at (81.3, 98.3)
- added D32: 1n4148, Diode_SMD:D_SOD-123, B.Cu at (100.3, 98.3)
- added D33: 1n4148, Diode_SMD:D_SOD-123, B.Cu at (119.4, 98.3)
- added D34: 1n4148, Diode_SMD:D_SOD-123, B.Cu at (197.8, 98.3)
- added D35: 1n4148, Diode_SMD:D_SOD-123, B.Cu at (216.8, 98.3)
- added D36: 1n4148, Diode_SMD:D_SOD-123, B.Cu at (235.9, 98.3)
- added D4: 1n4148, Diode_SMD:D_SOD-123, B.Cu at (100.3, 41.1)
- added D5: 1n4148, Diode_SMD:D_SOD-123, B.Cu at (119.4, 41.1)
- added D6: 1n4148, Diode_SMD:D_SOD-123, B.Cu at (197.8, 41.1)
- added D7: 1n4148, Diode_SMD:D_SOD-123, B.Cu at (216.8, 41.1)
- added D8: 1n4148, Diode_SMD:D_SOD-123, B.Cu at (235.9, 41.1)
- added D9: 1n4148, Diode_SMD:D_SOD-123, B.Cu at (254.9, 41.1)
- added MX1: SW, PCM_Switch_Keyboard_Cherry_MX:SW_Cherry_MX_PCB_1.00u, F.Cu at (38.1, 38.1)
- added MX10: SW, PCM_Switch_Keyboard_Cherry_MX:SW_Cherry_MX_PCB_1.00u, F.Cu at (268.9, 38.1)
- added MX11: SW, PCM_Switch_Keyboard_Cherry_MX:SW_Cherry_MX_PCB_1.00u, F.Cu at (38.1, 57.1)
- added MX12: SW, PCM_Switch_Keyboard_Cherry_MX:SW_Cherry_MX_PCB_1.00u, F.Cu at (57.1, 57.1)
- added MX13: SW, PCM_Switch_Keyboard_Cherry_MX:SW_Cherry_MX_PCB_1.00u, F.Cu at (76.2, 57.1)
- added MX14: SW, PCM_Switch_Keyboard_Cherry_MX:SW_Cherry_MX_PCB_1.00u, F.Cu at (95.2, 57.1)
- added MX15: SW, PCM_Switch_Keyboard_Cherry_MX:SW_Cherry_MX_PCB_1.00u, F.Cu at (114.3, 57.1)
- added MX16: SW, PCM_Switch_Keyboard_Cherry_MX:SW_Cherry_MX_PCB_1.00u, F.Cu at (192.7, 57.1)
- added MX17: SW, PCM_Switch_Keyboard_Cherry_MX:SW_Cherry_MX_PCB_1.00u, F.Cu at (211.7, 57.1)
- added MX18: SW, PCM_Switch_Keyboard_Cherry_MX:SW_Cherry_MX_PCB_1.00u, F.Cu at (230.8, 57.1)
- added MX19: SW, PCM_Switch_Keyboard_Cherry_MX:SW_Cherry_MX_PCB_1.00u, F.Cu at (249.8, 57.1)
- added MX2: SW, PCM_Switch_Keyboard_Cherry_MX:SW_Cherry_MX_PCB_1.00u, F.Cu at (57.1, 38.1)
- added MX20: SW, PCM_Switch_Keyboard_Cherry_MX:SW_Cherry_MX_PCB_1.00u, F.Cu at (268.9, 57.1)
- added MX21: SW, PCM_Switch_Keyboard_Cherry_MX:SW_Cherry_MX_PCB_1.00u, F.Cu at (38.1, 76.2)
- added MX22: SW, PCM_Switch_Keyboard_Cherry_MX:SW_Cherry_MX_PCB_1.00u, F.Cu at (57.1, 76.2)
- added MX23: SW, PCM_Switch_Keyboard_Cherry_MX:SW_Cherry_MX_PCB_1.00u, F.Cu at (76.2, 76.2)
- added MX24: SW, PCM_Switch_Keyboard_Cherry_MX:SW_Cherry_MX_PCB_1.00u, F.Cu at (95.2, 76.2)
- added MX25: SW, PCM_Switch_Keyboard_Cherry_MX:SW_Cherry_MX_PCB_1.00u, F.Cu at (114.3, 76.2)
- added MX26: SW, PCM_Switch_Keyboard_Cherry_MX:SW_Cherry_MX_PCB_1.00u, F.Cu at (192.7, 76.2)
- added MX27: SW, PCM_Switch_Keyboard_Cherry_MX:SW_Cherry_MX_PCB_1.00u, F.Cu at (211.7, 76.2)
- added MX28: SW, PCM_Switch_Keyboard_Cherry_MX:SW_Cherry_MX_PCB_1.00u, F.Cu at (230.8, 76.2)
- added MX29: SW, PCM_Switch_Keyboard_Cherry_MX:SW_Cherry_MX_PCB_1.00u, F.Cu at (249.8, 76.2)
- added MX3: SW, PCM_Switch_Keyboard_Cherry_MX:SW_Cherry_MX_PCB_1.00u, F.Cu at (76.2, 38.1)
- added MX30: SW, PCM_Switch_Keyboard_Cherry_MX:SW_Cherry_MX_PCB_1.00u, F.Cu at (268.9, 76.2)
- added MX31: SW, PCM_Switch_Keyboard_Cherry_MX:SW_Cherry_MX_PCB_1.00u, F.Cu at (76.2, 95.2)
- added MX32: SW, PCM_Switch_Keyboard_Cherry_MX:SW_Cherry_MX_PCB_1.00u, F.Cu at (95.2, 95.2)
- added MX33: SW, PCM_Switch_Keyboard_Cherry_MX:SW_Cherry_MX_PCB_1.00u, F.Cu at (114.3, 95.2)
- added MX34: SW, PCM_Switch_Keyboard_Cherry_MX:SW_Cherry_MX_PCB_1.00u, F.Cu at (192.7, 95.2)
- added MX35: SW, PCM_Switch_Keyboard_Cherry_MX:SW_Cherry_MX_PCB_1.00u, F.Cu at (211.7, 95.2)
- added MX36: SW, PCM_Switch_Keyboard_Cherry_MX:SW_Cherry_MX_PCB_1.00u, F.Cu at (230.8, 95.2)
- added MX4: SW, PCM_Switch_Keyboard_Cherry_MX:SW_Cherry_MX_PCB_1.00u, F.Cu at (95.2, 38.1)
- added MX5: SW, PCM_Switch_Keyboard_Cherry_MX:SW_Cherry_MX_PCB_1.00u, F.Cu at (114.3, 38.1)
- added MX6: SW, PCM_Switch_Keyboard_Cherry_MX:SW_Cherry_MX_PCB_1.00u, F.Cu at (192.7, 38.1)
- added MX7: SW, PCM_Switch_Keyboard_Cherry_MX:SW_Cherry_MX_PCB_1.00u, F.Cu at (211.7, 38.1)
- added MX8: SW, PCM_Switch_Keyboard_Cherry_MX:SW_Cherry_MX_PCB_1.00u, F.Cu at (230.8, 38.1)
- added MX9: SW, PCM_Switch_Keyboard_Cherry_MX:SW_Cherry_MX_PCB_1.00u, F.Cu at (249.8, 38.1)
Other:
- board outline added: 252.5 x 78.7 mm

Commit message: chore: minor updates
Parts:
- removed D1, D10, D11, D12, D13, D14, D15, D16, D17, D18, D19, D2, D20, D21, D22, D23, D24, D25, D26, D27, D28, D29, D3, D30, D31, D32, D33, D34, D35, D36, D4, D5, D6, D7, D8, D9: 1n4148, Diode_SMD:D_SOD-123
- removed MX1, MX10, MX11, MX12, MX13, MX14, MX15, MX16, MX17, MX18, MX19, MX2, MX20, MX21, MX22, MX23, MX24, MX25, MX26, MX27, MX28, MX29, MX3, MX30, MX31, MX32, MX33, MX34, MX35, MX36, MX4, MX5, MX6, MX7, MX8, MX9: SW, PCM_Switch_Keyboard_Cherry_MX:SW_Cherry_MX_PCB_1.00u
Other:
- board size 252.5 x 78.7 mm -> 28.8 x 41.8 mm
- board text added: "Break lines"
- board text added: "Switch (0,0)"

Commit message: Added keyboard_pad_left, keyboard_pad_right. Added LDOs, Added USB C connector. Added initial placement for keys.
Parts:
- added D1: 1n4148, Diode_SMD:D_SOD-123, B.Cu at (36.1, 31.1)
- added D10: 1n4148, Diode_SMD:D_SOD-123, B.Cu at (234.1, 30.9)
- added D11: 1n4148, Diode_SMD:D_SOD-123, B.Cu at (253.3, 30.9)
- added D12: 1n4148, Diode_SMD:D_SOD-123, B.Cu at (272.5, 30.9)
- added D13: 1n4148, Diode_SMD:D_SOD-123, B.Cu at (36.1, 50.3)
- added D14: 1n4148, Diode_SMD:D_SOD-123, B.Cu at (55.3, 50.3)
- added D15: 1n4148, Diode_SMD:D_SOD-123, B.Cu at (74.5, 50.3)
- added D16: 1n4148, Diode_SMD:D_SOD-123, B.Cu at (93.7, 50.3)
- added D17: 1n4148, Diode_SMD:D_SOD-123, B.Cu at (112.9, 50.3)
- added D18: 1n4148, Diode_SMD:D_SOD-123, B.Cu at (132.1, 50.3)
- added D19: 1n4148, Diode_SMD:D_SOD-123, B.Cu at (176.5, 50.1)
- added D2: 1n4148, Diode_SMD:D_SOD-123, B.Cu at (55.3, 31.1)
- added D20: 1n4148, Diode_SMD:D_SOD-123, B.Cu at (195.7, 50.1)
- added D21: 1n4148, Diode_SMD:D_SOD-123, B.Cu at (214.9, 50.1)
- added D22: 1n4148, Diode_SMD:D_SOD-123, B.Cu at (234.1, 50.1)
- added D23: 1n4148, Diode_SMD:D_SOD-123, B.Cu at (253.3, 50.1)
- added D24: 1n4148, Diode_SMD:D_SOD-123, B.Cu at (272.5, 50.1)
- added D25: 1n4148, Diode_SMD:D_SOD-123, B.Cu at (36.1, 69.5)
- added D26: 1n4148, Diode_SMD:D_SOD-123, B.Cu at (55.3, 69.5)
- added D27: 1n4148, Diode_SMD:D_SOD-123, B.Cu at (74.5, 69.5)
- added D28: 1n4148, Diode_SMD:D_SOD-123, B.Cu at (93.7, 69.5)
- added D29: 1n4148, Diode_SMD:D_SOD-123, B.Cu at (112.9, 69.5)
- added D3: 1n4148, Diode_SMD:D_SOD-123, B.Cu at (74.5, 31.1)
- added D30: 1n4148, Diode_SMD:D_SOD-123, B.Cu at (132.1, 69.5)
- added D31: 1n4148, Diode_SMD:D_SOD-123, B.Cu at (176.5, 69.3)
- added D32: 1n4148, Diode_SMD:D_SOD-123, B.Cu at (195.7, 69.3)
- added D33: 1n4148, Diode_SMD:D_SOD-123, B.Cu at (214.9, 69.3)
- added D34: 1n4148, Diode_SMD:D_SOD-123, B.Cu at (234.1, 69.3)
- added D35: 1n4148, Diode_SMD:D_SOD-123, B.Cu at (253.3, 69.3)
- added D36: 1n4148, Diode_SMD:D_SOD-123, B.Cu at (272.5, 69.3)
- added D37: 1n4148, Diode_SMD:D_SOD-123, B.Cu at (74.5, 88.7)
- added D38: 1n4148, Diode_SMD:D_SOD-123, B.Cu at (93.7, 88.7)
- added D39: 1n4148, Diode_SMD:D_SOD-123, B.Cu at (112.9, 88.7)
- added D4: 1n4148, Diode_SMD:D_SOD-123, B.Cu at (93.7, 31.1)
- added D40: 1n4148, Diode_SMD:D_SOD-123, B.Cu at (132.1, 88.7)
- added D41: 1n4148, Diode_SMD:D_SOD-123, B.Cu at (176.5, 88.5)
- added D42: 1n4148, Diode_SMD:D_SOD-123, B.Cu at (195.7, 88.5)
- added D43: 1n4148, Diode_SMD:D_SOD-123, B.Cu at (214.9, 88.5)
- added D44: 1n4148, Diode_SMD:D_SOD-123, B.Cu at (234.1, 88.5)
- added D5: 1n4148, Diode_SMD:D_SOD-123, B.Cu at (112.9, 31.1)
- added D6: 1n4148, Diode_SMD:D_SOD-123, B.Cu at (132.1, 31.1)
- added D7: 1n4148, Diode_SMD:D_SOD-123, B.Cu at (176.5, 30.9)
- added D8: 1n4148, Diode_SMD:D_SOD-123, B.Cu at (195.7, 30.9)
- added D9: 1n4148, Diode_SMD:D_SOD-123, B.Cu at (214.9, 30.9)
- added MX1: SW, PCM_Switch_Keyboard_Hotswap_Kailh:SW_Hotswap_Kailh_Choc_V1, F.Cu at (27.4, 27.9)
- added MX10: SW, PCM_Switch_Keyboard_Hotswap_Kailh:SW_Hotswap_Kailh_Choc_V1, F.Cu at (229.0, 27.9)
- added MX11: SW, PCM_Switch_Keyboard_Hotswap_Kailh:SW_Hotswap_Kailh_Choc_V1, F.Cu at (248.2, 27.9)
- added MX12: SW, PCM_Switch_Keyboard_Hotswap_Kailh:SW_Hotswap_Kailh_Choc_V1, F.Cu at (267.4, 27.9)
- added MX13: SW, PCM_Switch_Keyboard_Hotswap_Kailh:SW_Hotswap_Kailh_Choc_V1, F.Cu at (27.4, 47.1)
- added MX14: SW, PCM_Switch_Keyboard_Hotswap_Kailh:SW_Hotswap_Kailh_Choc_V1, F.Cu at (46.6, 47.1)
- added MX15: SW, PCM_Switch_Keyboard_Hotswap_Kailh:SW_Hotswap_Kailh_Choc_V1, F.Cu at (65.8, 47.1)
- added MX16: SW, PCM_Switch_Keyboard_Hotswap_Kailh:SW_Hotswap_Kailh_Choc_V1, F.Cu at (85.0, 47.1)
- added MX17: SW, PCM_Switch_Keyboard_Hotswap_Kailh:SW_Hotswap_Kailh_Choc_V1, F.Cu at (104.2, 47.1)
- added MX18: SW, PCM_Switch_Keyboard_Hotswap_Kailh:SW_Hotswap_Kailh_Choc_V1, F.Cu at (123.4, 47.1)
- added MX19: SW, PCM_Switch_Keyboard_Hotswap_Kailh:SW_Hotswap_Kailh_Choc_V1, F.Cu at (171.4, 47.1)
- added MX2: SW, PCM_Switch_Keyboard_Hotswap_Kailh:SW_Hotswap_Kailh_Choc_V1, F.Cu at (46.6, 27.9)
- added MX20: SW, PCM_Switch_Keyboard_Hotswap_Kailh:SW_Hotswap_Kailh_Choc_V1, F.Cu at (190.6, 47.1)
- added MX21: SW, PCM_Switch_Keyboard_Hotswap_Kailh:SW_Hotswap_Kailh_Choc_V1, F.Cu at (209.8, 47.1)
- added MX22: SW, PCM_Switch_Keyboard_Hotswap_Kailh:SW_Hotswap_Kailh_Choc_V1, F.Cu at (229.0, 47.1)
- added MX23: SW, PCM_Switch_Keyboard_Hotswap_Kailh:SW_Hotswap_Kailh_Choc_V1, F.Cu at (248.2, 47.1)
- added MX24: SW, PCM_Switch_Keyboard_Hotswap_Kailh:SW_Hotswap_Kailh_Choc_V1, F.Cu at (267.4, 47.1)
- added MX25: SW, PCM_Switch_Keyboard_Hotswap_Kailh:SW_Hotswap_Kailh_Choc_V1, F.Cu at (27.4, 66.3)
- added MX26: SW, PCM_Switch_Keyboard_Hotswap_Kailh:SW_Hotswap_Kailh_Choc_V1, F.Cu at (46.6, 66.3)
- added MX27: SW, PCM_Switch_Keyboard_Hotswap_Kailh:SW_Hotswap_Kailh_Choc_V1, F.Cu at (65.8, 66.3)
- added MX28: SW, PCM_Switch_Keyboard_Hotswap_Kailh:SW_Hotswap_Kailh_Choc_V1, F.Cu at (85.0, 66.3)
- added MX29: SW, PCM_Switch_Keyboard_Hotswap_Kailh:SW_Hotswap_Kailh_Choc_V1, F.Cu at (104.2, 66.3)
- added MX3: SW, PCM_Switch_Keyboard_Hotswap_Kailh:SW_Hotswap_Kailh_Choc_V1, F.Cu at (65.8, 27.9)
- added MX30: SW, PCM_Switch_Keyboard_Hotswap_Kailh:SW_Hotswap_Kailh_Choc_V1, F.Cu at (123.4, 66.3)
- added MX31: SW, PCM_Switch_Keyboard_Hotswap_Kailh:SW_Hotswap_Kailh_Choc_V1, F.Cu at (171.4, 66.3)
- added MX32: SW, PCM_Switch_Keyboard_Hotswap_Kailh:SW_Hotswap_Kailh_Choc_V1, F.Cu at (190.6, 66.3)
- added MX33: SW, PCM_Switch_Keyboard_Hotswap_Kailh:SW_Hotswap_Kailh_Choc_V1, F.Cu at (209.8, 66.3)
- added MX34: SW, PCM_Switch_Keyboard_Hotswap_Kailh:SW_Hotswap_Kailh_Choc_V1, F.Cu at (229.0, 66.3)
- added MX35: SW, PCM_Switch_Keyboard_Hotswap_Kailh:SW_Hotswap_Kailh_Choc_V1, F.Cu at (248.2, 66.3)
- added MX36: SW, PCM_Switch_Keyboard_Hotswap_Kailh:SW_Hotswap_Kailh_Choc_V1, F.Cu at (267.4, 66.3)
- added MX37: SW, PCM_Switch_Keyboard_Hotswap_Kailh:SW_Hotswap_Kailh_Choc_V1, F.Cu at (65.8, 85.5)
- added MX38: SW, PCM_Switch_Keyboard_Hotswap_Kailh:SW_Hotswap_Kailh_Choc_V1, F.Cu at (85.0, 85.5)
- added MX39: SW, PCM_Switch_Keyboard_Hotswap_Kailh:SW_Hotswap_Kailh_Choc_V1, F.Cu at (104.2, 85.5)
- added MX4: SW, PCM_Switch_Keyboard_Hotswap_Kailh:SW_Hotswap_Kailh_Choc_V1, F.Cu at (85.0, 27.9)
- added MX40: SW, PCM_Switch_Keyboard_Hotswap_Kailh:SW_Hotswap_Kailh_Choc_V1, F.Cu at (123.4, 85.5)
- added MX41: SW, PCM_Switch_Keyboard_Hotswap_Kailh:SW_Hotswap_Kailh_Choc_V1, F.Cu at (171.4, 85.5)
- added MX42: SW, PCM_Switch_Keyboard_Hotswap_Kailh:SW_Hotswap_Kailh_Choc_V1, F.Cu at (190.6, 85.5)
- added MX43: SW, PCM_Switch_Keyboard_Hotswap_Kailh:SW_Hotswap_Kailh_Choc_V1, F.Cu at (209.8, 85.5)
- added MX44: SW, PCM_Switch_Keyboard_Hotswap_Kailh:SW_Hotswap_Kailh_Choc_V1, F.Cu at (229.0, 85.5)
- added MX5: SW, PCM_Switch_Keyboard_Hotswap_Kailh:SW_Hotswap_Kailh_Choc_V1, F.Cu at (104.2, 27.9)
- added MX6: SW, PCM_Switch_Keyboard_Hotswap_Kailh:SW_Hotswap_Kailh_Choc_V1, F.Cu at (123.4, 27.9)
- added MX7: SW, PCM_Switch_Keyboard_Hotswap_Kailh:SW_Hotswap_Kailh_Choc_V1, F.Cu at (171.4, 27.9)
- added MX8: SW, PCM_Switch_Keyboard_Hotswap_Kailh:SW_Hotswap_Kailh_Choc_V1, F.Cu at (190.6, 27.9)
- added MX9: SW, PCM_Switch_Keyboard_Hotswap_Kailh:SW_Hotswap_Kailh_Choc_V1, F.Cu at (209.8, 27.9)
Other:
- board size 28.8 x 41.8 mm -> 262.2 x 79.8 mm
