File: hardware/b11/ecad/common/ETZ-B11-LLB.kicad_pcb (KiCad board)
At the start: 2 copper layers, 29 x 88.8 mm, 3 parts, among them J1 CN-HY04C-01D-MALE, J2 CN-HY04C-01D-FEMALE, J3 503480-2000

Commit message: feat: extend B11 carrier and logic board foundations
Signed-off-by: Nikola Secerovski <secersh@gmail.com>
Parts:
- J3: moved to B.Cu
- moved J3 0.87 mm to (139.2, 87.5), turned to 90 degrees
Other:
- outline, holes or cut-outs redrawn
