File: hardware/b11/ecad/common/ETZ-B11-RLB.kicad_pcb (KiCad board)
At the start: 2 copper layers, 29 x 88.8 mm, 2 parts, among them J1 CN-HY04C-01D-FEMALE, J2 CN-HY04C-01D-MALE

Commit message: feat: extend B11 carrier and logic board foundations
Signed-off-by: Nikola Secerovski <secersh@gmail.com>
Other:
- outline, holes or cut-outs redrawn
Changed lines of the file:
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@@
 	)
 	(gr_arc
-		(start 134 65.6)
-		(mid 135.464466 62.064466)
-		(end 139 60.6)
-		(stroke
-			(width 0.05)
-			(type default)
-		)
-		(layer "Edge.Cuts")
-	)
-	(gr_line
-		(start 161 110)
-		(end 163 110)
-		(stroke
-			(width 0.05)
-			(type default)
-		)
-		(layer "Edge.Cuts")
-	)
-	(gr_line
-		(start 139 149.4)
-		(end 158 149.4)
-		(stroke
-			(width 0.05)
-			(type default)
-		)
-		(layer "Edge.Cuts")
-	)
-	(gr_line
-		(start 163 110)
-		(end 163 144.4)
-		(stroke
-			(width 0.05)
-			(type default)
-		)
-		(layer "Edge.Cuts")
-	)
-	(gr_line
-		(start 163 80)
-		(end 161 79.999999)
-		(stroke
-			(width 0.05)
-			(type default)
-		)
-		(layer "Edge.Cuts")
-	)
-	(gr_line
-		(start 163 65.599999)
-		(end 163 80)
-		(stroke
-			(width 0.05)
-			(type default)
-		)
-		(layer "Edge.Cuts")
-	)
-	(gr_arc
-		(start 158 60.599999)
-		(mid 161.535534 62.064465)
-		(end 163 65.599999)
-		(stroke
-			(width 0.05)
-			(type default)
-		)
-		(layer "Edge.Cuts")
-	)
-	(gr_line
-		(start 159 82)
-		(end 159 108)
-		(stroke
-			(width 0.05)
-			(type default)
-		)
-		(layer "Edge.Cuts")
-	)
-	(gr_circle
-		(center 157.199999 145.2)
-		(end 158.649999 145.2)
-		(stroke
-			(width 0.05)
-			(type default)
-		)
-		(fill no)
-		(layer "Edge.Cuts")
-	)
-	(gr_arc
-		(start 163 144.4)
-		(mid 161.535534 147.935534)
-		(end 158 149.4)
-		(stroke
-			(width 0.05)
-			(type default)
-		)
-		(layer "Edge.Cuts")
-	)
-	(gr_circle
-		(center 157.199999 64.8)
-		(end 158.649999 64.8)
-		(stroke
-			(width 0.05)
-			(type default)
-		)
-		(fill no)
-		(layer "Edge.Cuts")
-	)
-	(gr_arc
-		(start 161 110)
-		(mid 159.585786 109.414214)
-		(end 159 108)
-		(stroke
-			(width 0.05)
-			(type default)
-		)
-		(layer "Edge.Cuts")
-	)
-	(gr_arc
-		(start 159 82)
-		(mid 159.585786 80.585786)
-		(end 161 80)
+		(start 161 95)
+		(mid 159.585786 94.414214)
+		(end 159 93)
 		(stroke
 			(width 0.05)
@@
 	)
 	(gr_line
-		(start 158 60.6)
-		(end 139 60.6)
+		(start 134 65.6)
+		(end 134 144.4)
+		(stroke
+			(width 0.05)
+			(type default)
+		)
+		(layer "Edge.Cuts")
+	)
+	(gr_arc
+		(start 158 60.599999)
+		(mid 161.535534 62.064465)
+		(end 163 65.599999)
+		(stroke
+			(width 0.05)
+			(type default)
+		)
+		(layer "Edge.Cuts")
+	)
+	(gr_arc
+		(start 159 82)
+		(mid 159.585786 80.585786)
+		(end 161 80)
 		(stroke
 			(width 0.05)
@@
 	)
 	(gr_line
-		(start 134 65.6)
-		(end 134 144.4)
+		(start 161 95)
+		(end 163 95)
+		(stroke
+			(width 0.05)
+			(type default)
+		)
+		(layer "Edge.Cuts")
+	)
+	(gr_circle
+		(center 157.199999 145.2)
+		(end 158.649999 145.2)
+		(stroke
+			(width 0.05)
+			(type default)
+		)
+		(fill no)
+		(layer "Edge.Cuts")
+	)
+	(gr_line
+		(start 159 82)
+		(end 159 93)
 		(stroke
 			(width 0.05)
@@
 		(layer "Edge.Cuts")
 	)
+	(gr_circle
+		(center 157.199999 64.8)
+		(end 158.649999 64.8)
+		(stroke
+			(width 0.05)
+			(type default)
+		)
+		(fill no)
+		(layer "Edge.Cuts")
+	)
+	(gr_line
+		(start 163 65.599999)
+		(end 163 80)
+		(stroke
+			(width 0.05)
+			(type default)
+		)
+		(layer "Edge.Cuts")
+	)
+	(gr_arc
+		(start 163 144.4)
+		(mid 161.535534 147.935534)
+		(end 158 149.4)
+		(stroke
+			(width 0.05)
+			(type default)
+		)
+		(layer "Edge.Cuts")
+	)
+	(gr_line
+		(start 158 60.6)
+		(end 139 60.6)
+		(stroke
+			(width 0.05)
+			(type default)
+		)
+		(layer "Edge.Cuts")
+	)
+	(gr_line
+		(start 139 149.4)
+		(end 158 149.4)
+		(stroke
+			(width 0.05)
+			(type default)
+		)
+		(layer "Edge.Cuts")
+	)
+	(gr_arc
+		(start 134 65.6)
+		(mid 135.464466 62.064466)
+		(end 139 60.6)
+		(stroke
+			(width 0.05)
+			(type default)
+		)
+		(layer "Edge.Cuts")
+	)
+	(gr_line
+		(start 163 95)
+		(end 163 144.4)
+		(stroke
+			(width 0.05)
+			(type default)
+		)
+		(layer "Edge.Cuts")
+	)
+	(gr_line
+		(start 163 80)
+		(end 161 80)
+		(stroke
+			(width 0.05)
+			(type default)
+		)
+		(layer "Edge.Cuts")
+	)
