File: hardware/b11/ecad/common/ETZ-B11-SP.kicad_sch (KiCad schematic)
At the start: 55 parts, among them J1 ETZ-B11-DSP

Commit message: feat: extend B11 carrier and logic board foundations
Signed-off-by: Nikola Secerovski <secersh@gmail.com>
Other:
- title: ETZ-B11-SP Common Switch Plate -> ETZ-B11-SP - Switch Plate
Changed lines of the file:
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@@
 	(paper "A2")
 	(title_block
-		(title "ETZ-B11-SP Common Switch Plate")
-		(rev "rev1")
+		(title "ETZ-B11-SP - Switch Plate")
+		(rev "1")
 		(company "etzee")
 	)
